File: 555-metronomo-1.kicad_pcb (KiCad board)
At the start: 2 copper layers, 10 parts, among them J1 Jack_3.5mm_3pin, J2 BARREL_JACK, U1 SE555

Commit message: dos layouts
Parts:
- moved RV1 45.9 mm to (108.1, 102.9)
- moved R1 37.1 mm to (161.4, 121.8), turned to 180 degrees
- moved J1 30.7 mm to (120.8, 116.8)
- moved C2 27.9 mm to (177.1, 102.0), turned to 180 degrees
- moved R2 26.4 mm to (161.4, 114.0), turned to 180 degrees
- moved J2 23.7 mm to (121.2, 132.3)
- moved U1 21.3 mm to (167.0, 113.8)
- moved D1 17.8 mm to (153.8, 115.6), turned to 270 degrees
- moved C3 17.2 mm to (137.9, 95.3)
- moved C1 16.7 mm to (177.7, 134.6), turned to 180 degrees
Routing:
- net Net-(C1-Pad2): track 0.00 -> 145.1 mm
- net RC-NET: track 95.9 -> 34.1 mm
- net DESC: track 29.9 -> 86.6 mm
- net Net-(R1-Pad2): track 23.8 -> 61.3 mm
- net GND: track 170.1 -> 142.0 mm
- net +BATT: track 10.2 -> 37.4 mm
- net Net-(C3-Pad1): track 12.3 -> 38.9 mm
- net Net-(J2-Pad3): track 26.5 -> 0.00 mm
- net V+: track 79.2 -> 56.6 mm
- net Net-(C3-Pad2): track 21.9 -> 31.2 mm
- added copper zone on B.Cu, net GND
- removed copper zone on F.Cu, net GND
Other:
- net class Default: clearance 0.2 -> 0.25; trace_width 0.25 -> 0.5
- net class power added: clearance 0.25, trace_width 0.8, via_dia 0.6, via_drill 0.4
- rule trace_clearance: 0.2 -> 0.25
