File: 555-metronomo.sch (KiCad schematic (older format))
At the start: 9 parts, among them U1 SE555

Commit message: .
Parts:
- C1, C2, C3: footprint (none) -> Capacitors_THT:CP_Axial_L34.5mm_D20.0mm_P41.00mm_Horizontal
- D1: footprint (none) -> Diodes_THT:D_DO-41_SOD81_P5.08mm_Vertical_AnodeUp
Changed lines of the file:
@@
 LIBS:contrib
 LIBS:valves
+LIBS:555-metronomo-cache
 EELAYER 25 0
 EELAYER END
@@
 F 0 "D1" H 2200 2650 50  0000 C CNN
 F 1 "1N4001" H 2200 2450 50  0000 C CNN
-F 2 "" H 2200 2550 50  0001 C CNN
+F 2 "Diodes_THT:D_DO-41_SOD81_P5.08mm_Vertical_AnodeUp" H 2200 2550 50  0001 C CNN
 F 3 "" H 2200 2550 50  0001 C CNN
 	1    2200 2550
@@
 F 0 "C3" H 4625 3700 50  0000 L CNN
 F 1 "100uF" H 4625 3500 50  0000 L CNN
-F 2 "" H 4638 3450 50  0001 C CNN
+F 2 "Capacitors_THT:CP_Axial_L34.5mm_D20.0mm_P41.00mm_Horizontal" H 4638 3450 50  0001 C CNN
 F 3 "" H 4600 3600 50  0001 C CNN
 	1    4600 3600
@@
 F 0 "C1" H 2225 4300 50  0000 L CNN
 F 1 "2uF" H 2225 4100 50  0000 L CNN
-F 2 "" H 2238 4050 50  0001 C CNN
+F 2 "Capacitors_THT:CP_Axial_L34.5mm_D20.0mm_P41.00mm_Horizontal" H 2238 4050 50  0001 C CNN
 F 3 "" H 2200 4200 50  0001 C CNN
 	1    2200 4200
@@
 F 0 "C2" H 2225 4600 50  0000 L CNN
 F 1 "2uF" H 2225 4400 50  0000 L CNN
-F 2 "" H 2238 4350 50  0001 C CNN
+F 2 "Capacitors_THT:CP_Axial_L34.5mm_D20.0mm_P41.00mm_Horizontal" H 2238 4350 50  0001 C CNN
 F 3 "" H 2200 4500 50  0001 C CNN
 	1    2200 4500

Commit message: dos layouts
Parts:
- removed LS1: Speaker, symbol Speaker
- added J1: Jack_3.5mm_3pin, Connectors:BARREL_JACK, symbol Jack_3.5mm_3pin
- added J2: BARREL_JACK, Connectors:BARREL_JACK, symbol BARREL_JACK
- C1, C2: footprint Capacitors_THT:CP_Axial_L34.5mm_D20.0mm_P41.00mm_Horizontal -> Capacitors_THT:CP_Axial_L18.0mm_D6.5mm_P25.00mm_Horizontal
- R1, R2: footprint (none) -> Resistors_THT:R_Axial_DIN0204_L3.6mm_D1.6mm_P1.90mm_Vertical
- RV1: footprint (none) -> Potentiometers:Potentiometer_Alps_RK09K_Horizontal
- U1: footprint (none) -> Housings_DIP:DIP-8_W7.62mm
Connections:
- net +BATT: now also J2.1
- net GND: now also J1.1 (S), J2.2
- net at C3.2: now also J1.3 (R)
- no-connect marks 1 -> 3
Other:
- moved on the sheet: C1, C2, C3, D1, R1, R2, RV1, U1
